File: pcb/DronePwrCut.brd (EAGLE design)
At the start: 82.5 x 35.5 mm, 55 parts, among them IC1 ATMega48, IC2 MIC5219-3.6YM5-TR, M1 AUIRFS8409-7P, M2 AUIRFS8409-7P, M3 AUIRFS8409-7P, M4 AUIRFS8409-7P, Q1 NF, X1 ISP

Commit message: Change resistor values (R2, R8) to handle low voltage (3V3) input signals correctly
Parts:
- R2: value 10k -> 4k7
- R8: value 20k -> 40k2
Changed lines of the file:
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@@
 <attribute name="NAME" x="10.4775" y="24.765" size="1.016" layer="25" font="vector" rot="R90"/>
 </element>
-<element name="R2" library="rcl" package="R1206" value="10k" x="9.2075" y="17.145" smashed="yes">
+<element name="R2" library="rcl" package="R1206" value="4k7" x="9.2075" y="17.145" smashed="yes">
 <attribute name="NAME" x="9.2075" y="18.0975" size="1.016" layer="25" font="vector"/>
 </element>
@@
 <attribute name="VALUE" x="67.945" y="30.445" size="0.0254" layer="27"/>
 </element>
-<element name="R8" library="rcl" package="R1206" value="20k" x="12.065" y="13.335" smashed="yes" rot="R90">
+<element name="R8" library="rcl" package="R1206" value="40k2" x="12.065" y="13.335" smashed="yes" rot="R90">
 <attribute name="NAME" x="13.335" y="14.605" size="1.016" layer="25" font="vector" rot="R270"/>
 </element>
